File: cirrata_pcb.kicad_sch (KiCad schematic)
At the start: 0 parts

Commit message: adicionando hierarquia nos arquivos do kicad para power, esp_32 e lora... movendo todos os códigos pra dentro da pasta "src"
Other:
- added sheet esp_32 (esp32_circuit.kicad_sch)
- added sheet lora_transceiver (lora_transceiver.kicad_sch)
- added sheet power (power.kicad_sch)
Changed lines of the file:
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@@
 	(generator_version "9.0")
 	(paper "A4")
+	(sheet
+		(at 137.16 31.75)
+		(size 33.02 27.94)
+		(exclude_from_sim no)
+		(in_bom yes)
+		(on_board yes)
+		(dnp no)
+		(fields_autoplaced yes)
+		(stroke
+			(width 0.1524)
+			(type solid)
+		)
+		(fill
+			(color 0 0 0 0.0000)
+		)
+		(property "Sheetname" "lora_transceiver"
+			(at 137.16 31.0384 0)
+			(effects
+				(font
+					(size 1.27 1.27)
+				)
+				(justify left bottom)
+			)
+		)
+		(property "Sheetfile" "lora_transceiver.kicad_sch"
+			(at 137.16 60.2746 0)
+			(effects
+				(font
+					(size 1.27 1.27)
+				)
+				(justify left top)
+			)
+		)
+		(instances
+			(project "cirrata_pcb"
+				(path "/ef8082a7-51b7-4699-9341-b4a68179aab4"
+					(page "4")
+				)
+			)
+		)
+	)
+	(sheet
+		(at 33.02 31.75)
+		(size 33.02 27.94)
+		(exclude_from_sim no)
+		(in_bom yes)
+		(on_board yes)
+		(dnp no)
+		(fields_autoplaced yes)
+		(stroke
+			(width 0.1524)
+			(type solid)
+		)
+		(fill
+			(color 0 0 0 0.0000)
+		)
+		(property "Sheetname" "power"
+			(at 33.02 31.0384 0)
+			(effects
+				(font
+					(size 1.27 1.27)
+				)
+				(justify left bottom)
+			)
+		)
+		(property "Sheetfile" "power.kicad_sch"
+			(at 33.02 60.2746 0)
+			(effects
+				(font
+					(size 1.27 1.27)
+				)
+				(justify left top)
+			)
+		)
+		(instances
+			(project "cirrata_pcb"
+				(path "/ef8082a7-51b7-4699-9341-b4a68179aab4"
+					(page "2")
+				)
+			)
+		)
+	)
+	(sheet
+		(at 83.82 31.75)
+		(size 33.02 27.94)
+		(exclude_from_sim no)
+		(in_bom yes)
+		(on_board yes)
+		(dnp no)
+		(fields_autoplaced yes)
+		(stroke
+			(width 0.1524)
+			(type solid)
+		)
+		(fill
+			(color 0 0 0 0.0000)
+		)
+		(property "Sheetname" "esp_32"
+			(at 83.82 31.0384 0)
+			(effects
+				(font
+					(size 1.27 1.27)
+				)
+				(justify left bottom)
+			)
+		)
+		(property "Sheetfile" "esp32_circuit.kicad_sch"
+			(at 83.82 60.2746 0)
+			(effects
+				(font
+					(size 1.27 1.27)
+				)
+				(justify left top)
+			)
+		)
+		(instances
+			(project "cirrata_pcb"
+				(path "/ef8082a7-51b7-4699-9341-b4a68179aab4"
+					(page "3")
+				)
+			)
+		)
+	)
 	(sheet_instances
 		(path "/"
